File: docs/KiCad/SmartThermostat.sch (KiCad schematic (older format))
At the start: 24 parts, among them U1 AMS1117-3.3, U2 ESP-8266, U4 DS18B20

Commit message: Updated documentation
Parts:
- removed D1: DIODE, ~, symbol DIODE
- removed R6: R, ~, symbol R
- removed RL1: Relay, symbol FINDER-36.11.4001
- removed U?: Opto transistor, ~, symbol PHDARL
- added D?: DIODE, ~, symbol DIODE
- added K1: SSR, ~, symbol SX12S01
- added Q?: 2N3904, ~, symbol NPN
- added R8: 1k, ~, symbol R
- added R9, R? (x2): 1.47k, ~, symbol R
- added R?: 4.7k, ~, symbol R
- added R?: 200, ~, symbol R
- added RL?: Relay, symbol FINDER-36.11.4001
- added To? (x2): CONN_1, ~, symbol CONN_1
- added U?: ESP-8266, symbol ESP-01V090
- added U?: DS18B20, symbol DS18B20
- added U?: Opto transistor, ~, symbol PHDARL
- renumbered 5V to 5V~OUT, To to To~Monitor~RX, To to To~Monitor~TX, To to To~Prog~RX, To to To~Prog~TX
Connections:
- wire segments 40 -> 65
Other:
- note added: "Execution mode (active high 5v)"
- note added: "Execution mode (active low 3.3v)"
- note removed: "Execution mode"
- moved on the sheet: 5V OUT, To Monitor RX, To Monitor TX, To Prog RX, To Prog TX
